Commit message: Removed claw r and l joints from rmpflow config to allow control outside of it.

File: extension/Autonomous_forwarder_python/motion_policy_configs/dev_forwarder_arm.urdf (robot description, URDF)
Before this commit: robot dev_forwarder_arm, 28 links, 27 joints
Links:
- link bunk: geometry collision mesh filename=meshes/bunk_vis.obj scale=1. 1. 1.; visual mesh filename=meshes/bunk_vis.obj scale=1. 1. 1.
- link crane_arm1: geometry collision mesh filename=meshes/crane_arm1_arm1.obj scale=1. 1. 1.; visual mesh filename=meshes/crane_arm1_arm1.obj scale=1. 1. 1.
- link crane_arm1_piston: geometry collision mesh filename=meshes/crane_arm1_piston_arm1_piston.obj scale=1. 1. 1.; visual mesh filename=meshes/crane_arm1_piston_arm1_piston.obj scale=1. 1. 1.
- link crane_arm1_piston_rod: geometry collision mesh filename=meshes/crane_arm1_piston_rod_arm1_piston_rod.obj scale=1. 1. 1.; visual mesh filename=meshes/crane_arm1_piston_rod_arm1_piston_rod.obj scale=1. 1. 1.
- link crane_arm2: geometry collision mesh filename=meshes/crane_arm2_arm2.obj scale=1. 1. 1.; visual mesh filename=meshes/crane_arm2_arm2.obj scale=1. 1. 1.
- link crane_arm2_linkage: geometry collision mesh filename=meshes/crane_arm2_linkage_arm2_linkage.obj scale=1. 1. 1.; visual mesh filename=meshes/crane_arm2_linkage_arm2_linkage.obj scale=1. 1. 1.
- link crane_arm2_piston: geometry collision mesh filename=meshes/crane_arm2_piston_arm2_piston.obj scale=1. 1. 1.; visual mesh filename=meshes/crane_arm2_piston_arm2_piston.obj scale=1. 1. 1.
- link crane_arm2_piston_rod: geometry collision mesh filename=meshes/crane_arm2_piston_rod_arm2_piston_rod.obj scale=1. 1. 1.; visual mesh filename=meshes/crane_arm2_piston_rod_arm2_piston_rod.obj scale=1. 1. 1.
- link crane_arm3: geometry collision mesh filename=meshes/crane_arm3_arm3.obj scale=1. 1. 1.; visual mesh filename=meshes/crane_arm3_arm3.obj scale=1. 1. 1.
- link crane_arm3_linkage: geometry collision mesh filename=meshes/crane_arm3_linkage_arm3_linkage.obj scale=1. 1. 1.; visual mesh filename=meshes/crane_arm3_linkage_arm3_linkage.obj scale=1. 1. 1.
- link crane_arm3_piston: geometry collision mesh filename=meshes/crane_arm3_piston_arm3_piston.obj scale=1. 1. 1.; visual mesh filename=meshes/crane_arm3_piston_arm3_piston.obj scale=1. 1. 1.
- link crane_arm3_piston_rod: geometry collision mesh filename=meshes/crane_arm3_piston_rod_arm3_piston_rod.obj scale=1. 1. 1.; visual mesh filename=meshes/crane_arm3_piston_rod_arm3_piston_rod.obj scale=1. 1. 1.
- link crane_arm4: geometry collision mesh filename=meshes/crane_arm4_arm4.obj scale=1. 1. 1.; visual mesh filename=meshes/crane_arm4_arm4.obj scale=1. 1. 1.
- link crane_arm5: geometry collision mesh filename=meshes/crane_arm5_arm5.obj scale=1. 1. 1.; visual mesh filename=meshes/crane_arm5_arm5.obj scale=1. 1. 1.
- link crane_base: geometry collision mesh filename=meshes/crane_base_base.obj scale=1. 1. 1.; visual mesh filename=meshes/crane_base_base.obj scale=1. 1. 1.
- link crane_claw_left: geometry collision mesh filename=meshes/crane_claw_left_claw_left.obj scale=1. 1. 1.; visual mesh filename=meshes/crane_claw_left_claw_left.obj scale=1. 1. 1.
- link crane_claw_piston: geometry collision mesh filename=meshes/crane_claw_piston_claw_piston.obj scale=1. 1. 1.; visual mesh filename=meshes/crane_claw_piston_claw_piston.obj scale=1. 1. 1.
- link crane_claw_piston_rod: geometry collision mesh filename=meshes/crane_claw_piston_rod_claw_piston_rod.obj scale=1. 1. 1.; visual mesh filename=meshes/crane_claw_piston_rod_claw_piston_rod.obj scale=1. 1. 1.
- link crane_claw_right: geometry collision mesh filename=meshes/crane_claw_right_claw_right.obj scale=1. 1. 1.; visual mesh filename=meshes/crane_claw_right_claw_right.obj scale=1. 1. 1.
- link crane_claw_x_rot: geometry collision mesh filename=meshes/crane_claw_x_rot_claw_x_rot.obj scale=1. 1. 1.; visual mesh filename=meshes/crane_claw_x_rot_claw_x_rot.obj scale=1. 1. 1.
- link crane_claw_y_rot: geometry collision mesh filename=meshes/crane_claw_y_rot_claw_y_rot.obj scale=1. 1. 1.; visual mesh filename=meshes/crane_claw_y_rot_claw_y_rot.obj scale=1. 1. 1.
- link crane_claw_z_rot: geometry collision mesh filename=meshes/crane_claw_z_rot_claw_z_rot.obj scale=1. 1. 1.; visual mesh filename=meshes/crane_claw_z_rot_claw_z_rot.obj scale=1. 1. 1.

Commit message: rmpflow config files

File: extension/Autonomous_forwarder_python/motion_policy_configs/dev_forwarder_arm.urdf (robot description, URDF)
Before this commit: robot dev_forwarder_arm, 28 links, 27 joints
Links:
- added link arm_end_effector
Joints:
- added joint crane_arm_end_effector_arm_end_effector: type fixed, parent crane_claw_z_rot, child arm_end_effector, origin xyz=0. -0.0000059 -0.606272  rpy=-0. 0. 0.
- joint a1_joint: limit lower=-2.6179939 upper=2.6179939 effort=200. velocity=0. -> lower=-2.6179939 upper=2.6179939 effort=200. velocity=10
- joint a1_piston_rod_prisjoint: limit lower=-inf upper=inf effort=0. velocity=0. -> lower=-360 upper=360 effort=0. velocity=10
- joint a2__joint: limit lower=-0.3665191 upper=1.0471976 effort=350. velocity=0. -> lower=-0.3665191 upper=1.0471976 effort=350. velocity=10
- joint a2_piston_rod_prisjoint: limit lower=-inf upper=inf effort=0. velocity=0. -> lower=-360 upper=360 effort=0. velocity=10
- joint a3_joint: limit lower=-2.7925268 upper=0.0872665 effort=200. velocity=0. -> lower=-2.7925268 upper=0.0872665 effort=200. velocity=10
- joint a3_piston_prisjoint: limit lower=-inf upper=inf effort=0. velocity=0. -> lower=-360 upper=360 effort=0. velocity=10
- joint a4_joint: limit lower=0. upper=2.2 effort=300. velocity=0. -> lower=0. upper=2.2 effort=300. velocity=10
- joint a5_joint: limit lower=-inf upper=inf effort=inf velocity=0. -> lower=-360 upper=360 effort=360 velocity=10
- joint claw_l_joint: limit lower=0. upper=2.5307274 effort=inf velocity=0. -> lower=0. upper=2.5307274 effort=360 velocity=10
- joint claw_piston_rod_prisjoint: limit lower=-inf upper=inf effort=0. velocity=0. -> lower=-360 upper=360 effort=0. velocity=10
- joint claw_r_joint: limit lower=0. upper=2.5307274 effort=0.1 velocity=0. -> lower=0. upper=2.5307274 effort=0.1 velocity=10
- joint claw_z_joint: limit (none) -> lower=-6.2831853 upper=6.2831853 effort=3. velocity=10.; type continuous -> revolute
